File: Pixy-mega128-0-sdram-hat/Pixy-mega128-0-sdram-hat.kicad_sch (KiCad schematic)
At the start: 9 parts, among them J1 PA_Header, J2 PB_Header, J3 PC_Header, J4 PD_Header, J5 PE_Header, J6 PF_Header, J8 Power_Header, U1 EDS1216AGTA

Commit message: Fixed lacking C3.
Parts:
- added C3: 0.1u, kekyo:C_Disc_D4.3mm_W1.9mm_P5.00mm, symbol kekyo:C
Connections:
- net GND: now also C3.2
- net VCC: now also C3.1
Changed lines of the file:
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@@
 (kicad_sch (version 20230121) (generator eeschema)
   (paper "A4")
+  (junction (at 59.69 146.05) (diameter 0) (color 0 0 0 0)
+  )
+  (junction (at 59.69 163.83) (diameter 0) (color 0 0 0 0)
+  )
   (junction (at 107.95 119.38) (diameter 0) (color 0 0 0 0)
   )
@@
     (stroke (width 0) (type default))
   )
+  (wire (pts (xy 59.69 163.83) (xy 72.39 163.83))
+    (stroke (width 0) (type default))
+  )
   (wire (pts (xy 195.58 105.41) (xy 203.2 105.41))
     (stroke (width 0) (type default))
@@
     (stroke (width 0) (type default))
   )
+  (wire (pts (xy 59.69 146.05) (xy 72.39 146.05))
+    (stroke (width 0) (type default))
+  )
   (bus (pts (xy 205.74 130.81) (xy 205.74 133.35))
     (stroke (width 0) (type default))
@@
     (stroke (width 0) (type default))
   )
+  (wire (pts (xy 72.39 146.05) (xy 72.39 151.13))
+    (stroke (width 0) (type default))
+  )
   (wire (pts (xy 41.91 154.94) (xy 48.26 154.94))
     (stroke (width 0) (type default))
@@
   )
   (bus (pts (xy 121.92 53.34) (xy 121.92 58.42))
+    (stroke (width 0) (type default))
+  )
+  (wire (pts (xy 72.39 158.75) (xy 72.39 163.83))
     (stroke (width 0) (type default))
   )
@@
         )
       )
+    )
+  )
+  (symbol (lib_name "C_1") (lib_id "kekyo:C") (at 72.39 154.94 0) (unit 1)
+    (in_bom yes) (on_board yes) (dnp no) (fields_autoplaced)
+    (property "Reference" "C3" (at 76.2 153.67 0)
+      (effects (font (size 1.27 1.27)) (justify left))
+    )
+    (property "Value" "0.1u" (at 76.2 156.21 0)
+      (effects (font (size 1.27 1.27)) (justify left))
+    )
+    (property "Footprint" "kekyo:C_Disc_D4.3mm_W1.9mm_P5.00mm" (at 73.3552 158.75 0)
+      (effects (font (size 1.27 1.27)) hide)
+    )
+    (property "Datasheet" "~" (at 72.39 154.94 0)
+      (effects (font (size 1.27 1.27)) hide)
+    )
+    (pin "1")
+    (pin "2")
+    (instances
+      (project "Pixy-mega128-0-sdram-hat"
+        (path "/75eb9fb0-9cf3-4dbf-ba78-916956d56cb1"
+          (reference "C3") (unit 1)
+        )
+      )
+      (project "Pixy-mega128"
+        (path "/7609de31-cb73-4ace-8f34-65caa63c74e9"
+          (reference "C5") (unit 1)
+        )
+      )
+      (project "MC68SEC000"
+        (path "/7907391b-035a-42ea-89b1-82b781ee98c8"
+          (reference "C1") (unit 1)
+        )
+      )
