File: Pixy-68000/KiCad/Pixy-68000.kicad_sch (KiCad schematic)
At the start: 92 parts, among them J1 AVR_ISP, J10 Header3, J11 USB, J4 Socket5, J5 Socket5, J6 JTAG, J6 Socket5, J7 Socket5, J8 BUS, J9 Header8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

Commit message: Added errara2 information.
Fixed missing SPISS signal.
Parts:
- removed J10: Header3, kekyo:PinHeader_1x03_P2.54mm_Vertical, symbol kekyo:Header3
- added J11: SPI, kekyo:PinSocket_1x05_P2.54mm_Vertical, symbol kekyo:Socket5
- added J12: CPUSIGNAL, kekyo:PinHeader_2x03_P2.54mm_Vertical, symbol kekyo:Socket2x3
Connections:
- net CPUCLK: now also J12.1 (P0)
- net GND: now also J11.5 (P4)
- net SPICLK: now also J11.1 (P0)
- net SPISI: now also J11.2 (P1)
- net SPISO: now also J11.3 (P2)
- net /BERR: now also J12.6 (P5)
- net /BG: now also J12.5 (P4)
- net /BR: now also J12.3 (P2)
- net /HALT: now also J12.4 (P3)
- net /RESET: now also J12.2 (P1)
- net /SW2: now also U5.8 (XTAL2/PB7); no longer U5.14 (PB2)
- net /SPISS: now reaches U4.82 (PT10C/JTAGENB)
- net /SPISS: now also U5.14 (PB2), J11.4 (P3)
Other:
- moved on the sheet: J9

Commit message: Totally checked booting from flash rom.
Connections:
- net /PROMCS0: now also R15.2, U10.22 (CE), U4.30 (PB4D); no longer R14.2, U11.22 (CE), U4.29 (PB4C)
- net /PROMCS1: now also R14.2, U11.22 (CE), U4.29 (PB4C); no longer R15.2, U10.22 (CE), U4.30 (PB4D)
- net /SRAMCS0: now also R15.2, U4.28 (PB4B), U6.8 (~{CE}); no longer R14.2, U4.27 (PB4A/CSSPIN), U7.8 (~{CE})
- net /SRAMCS1: now also R14.2, U4.27 (PB4A/CSSPIN), U7.8 (~{CE}); no longer R15.2, U4.28 (PB4B), U6.8 (~{CE})
Changed lines of the file:
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@@
+    (effects (font (size 1.27 1.27)) (justify left bottom))
+  )
+  (label "{slash}SRAMCS1" (at 391.16 160.02 0) (fields_autoplaced)
     (effects (font (size 1.27 1.27)) (justify left bottom))
   )
@@
     (effects (font (size 1.27 1.27)) (justify left bottom))
   )
-  (label "{slash}SRAMCS0" (at 391.16 160.02 0) (fields_autoplaced)
-    (effects (font (size 1.27 1.27)) (justify left bottom))
-  )
-  (label "{slash}PROMCS0" (at 360.68 93.98 90) (fields_autoplaced)
-    (effects (font (size 1.27 1.27)) (justify left bottom))
-  )
   (label "RUN" (at 105.41 93.98 90) (fields_autoplaced)
     (effects (font (size 1.27 1.27)) (justify left bottom))
@@
     (effects (font (size 1.27 1.27)) (justify left bottom))
   )
+  (label "{slash}PROMCS1" (at 499.11 167.64 0) (fields_autoplaced)
+    (effects (font (size 1.27 1.27)) (justify left bottom))
+  )
   (label "A15" (at 132.08 161.29 0) (fields_autoplaced)
     (effects (font (size 1.27 1.27)) (justify left bottom))
@@
     (effects (font (size 1.27 1.27)) (justify left bottom))
   )
-  (label "{slash}SRAMCS0" (at 347.98 93.98 90) (fields_autoplaced)
-    (effects (font (size 1.27 1.27)) (justify left bottom))
-  )
   (label "D8" (at 434.34 109.22 0) (fields_autoplaced)
     (effects (font (size 1.27 1.27)) (justify left bottom))
@@
     (effects (font (size 1.27 1.27)) (justify left bottom))
   )
+  (label "{slash}PROMCS1" (at 360.68 93.98 90) (fields_autoplaced)
+    (effects (font (size 1.27 1.27)) (justify left bottom))
+  )
   (label "A13" (at 441.96 142.24 0) (fields_autoplaced)
     (effects (font (size 1.27 1.27)) (justify left bottom))
@@
     (effects (font (size 1.27 1.27)) (justify left bottom))
   )
-  (label "{slash}PROMCS1" (at 441.96 167.64 0) (fields_autoplaced)
-    (effects (font (size 1.27 1.27)) (justify left bottom))
-  )
   (label "A9" (at 441.96 132.08 0) (fields_autoplaced)
     (effects (font (size 1.27 1.27)) (justify left bottom))
   )
-  (label "{slash}SRAMCS1" (at 340.36 160.02 0) (fields_autoplaced)
-    (effects (font (size 1.27 1.27)) (justify left bottom))
-  )
   (label "A7" (at 547.37 227.33 0) (fields_autoplaced)
     (effects (font (size 1.27 1.27)) (justify left bottom))
@@
     (effects (font (size 1.27 1.27)) (justify left bottom))
   )
-  (label "{slash}SRAMCS1" (at 184.15 177.8 0) (fields_autoplaced)
-    (effects (font (size 1.27 1.27)) (justify left bottom))
-  )
   (label "D4" (at 304.8 154.94 0) (fields_autoplaced)
     (effects (font (size 1.27 1.27)) (justify left bottom))
@@
     (effects (font (size 1.27 1.27)) (justify left bottom))
   )
+  (label "{slash}PROMCS0" (at 184.15 182.88 0) (fields_autoplaced)
+    (effects (font (size 1.27 1.27)) (justify left bottom))
+  )
   (label "A7" (at 184.15 215.9 0) (fields_autoplaced)
     (effects (font (size 1.27 1.27)) (justify left bottom))
@@
     (effects (font (size 1.27 1.27)) (justify left bottom))
   )
+  (label "{slash}PROMCS0" (at 441.96 167.64 0) (fields_autoplaced)
+    (effects (font (size 1.27 1.27)) (justify left bottom))
+  )
   (label "{slash}STEPEN" (at 68.58 93.98 90) (fields_autoplaced)
     (effects (font (size 1.27 1.27)) (justify left bottom))
@@
     (effects (font (size 1.27 1.27)) (justify left bottom))
   )
-  (label "{slash}SRAMCS1" (at 354.33 93.98 90) (fields_autoplaced)
-    (effects (font (size 1.27 1.27)) (justify left bottom))
-  )
   (label "{slash}IPL2" (at 63.5 135.89 0) (fields_autoplaced)
     (effects (font (size 1.27 1.27)) (justify left bottom))
@@
     (effects (font (size 1.27 1.27)) (justify left bottom))
   )
+  (label "{slash}SRAMCS1" (at 347.98 93.98 90) (fields_autoplaced)
+    (effects (font (size 1.27 1.27)) (justify left bottom))
+  )
   (label "MCLK" (at 335.28 93.98 90) (fields_autoplaced)
     (effects (font (size 1.27 1.27)) (justify left bottom))
@@
     (effects (font (size 1.27 1.27)) (justify left bottom))
   )
-  (label "{slash}SRAMCS0" (at 184.15 175.26 0) (fields_autoplaced)
-    (effects (font (size 1.27 1.27)) (justify left bottom))
-  )
   (label "LEDDIO1" (at 299.72 327.66 0) (fields_autoplaced)
     (effects (font (size 1.27 1.27)) (justify left bottom))
@@
     (effects (font (size 1.27 1.27)) (justify left bottom))
   )
-  (label "{slash}PROMCS0" (at 184.15 180.34 0) (fields_autoplaced)
-    (effects (font (size 1.27 1.27)) (justify left bottom))
-  )
   (label "A12" (at 441.96 139.7 0) (fields_autoplaced)
     (effects (font (size 1.27 1.27)) (justify left bottom))
@@
     (effects (font (size 1.27 1.27)) (justify left bottom))
   )
+  (label "{slash}PROMCS1" (at 184.15 180.34 0) (fields_autoplaced)
+    (effects (font (size 1.27 1.27)) (justify left bottom))
+  )
   (label "A22" (at 303.53 208.28 0) (fields_autoplaced)
     (effects (font (size 1.27 1.27)) (justify left bottom))
@@
     (effects (font (size 1.27 1.27)) (justify left bottom))
   )
+  (label "{slash}SRAMCS0" (at 354.33 93.98 90) (fields_autoplaced)
+    (effects (font (size 1.27 1.27)) (justify left bottom))
+  )
   (label "{slash}AVEC" (at 184.15 147.32 0) (fields_autoplaced)
     (effects (font (size 1.27 1.27)) (justify left bottom))
@@
     (effects (font (size 1.27 1.27)) (justify left bottom))
   )
+  (label "{slash}PROMCS0" (at 367.03 93.98 90) (fields_autoplaced)
+    (effects (font (size 1.27 1.27)) (justify left bottom))
+  )
   (label "A2" (at 499.11 114.3 0) (fields_autoplaced)
     (effects (font (size 1.27 1.27)) (justify left bottom))
@@
     (effects (font (size 1.27 1.27)) (justify left bottom))
   )
-  (label "{slash}PROMCS1" (at 184.15 182.88 0) (fields_autoplaced)
-    (effects (font (size 1.27 1.27)) (justify left bottom))
-  )
   (label "A14" (at 184.15 243.84 0) (fields_autoplaced)
     (effects (font (size 1.27 1.27)) (justify left bottom))
@@
     (effects (font (size 1.27 1.27)) (justify left bottom))
   )
-  (label "{slash}PROMCS1" (at 367.03 93.98 90) (fields_autoplaced)
+  (label "{slash}SRAMCS0" (at 340.36 160.02 0) (fields_autoplaced)
     (effects (font (size 1.27 1.27)) (justify left bottom))
   )
@@
     (effects (font (size 1.27 1.27)) (justify left bottom))
   )
-  (label "{slash}PROMCS0" (at 499.11 167.64 0) (fields_autoplaced)
-    (effects (font (size 1.27 1.27)) (justify left bottom))
-  )
   (label "D11" (at 499.11 237.49 0) (fields_autoplaced)
     (effects (font (size 1.27 1.27)) (justify left bottom))
@@
     (effects (font (size 1.27 1.27)) (justify left bottom))
   )
+  (label "{slash}SRAMCS0" (at 184.15 177.8 0) (fields_autoplaced)
+    (effects (font (size 1.27 1.27)) (justify left bottom))
+  )
   (label "{slash}BERR" (at 544.83 295.91 0) (fields_autoplaced)
     (effects (font (size 1.27 1.27)) (justify left bottom))
@@
     (effects (font (size 1.27 1.27)) (justify left bottom))
   )
+  (label "{slash}SRAMCS1" (at 184.15 175.26 0) (fields_autoplaced)
+    (effects (font (size 1.27 1.27)) (justify left bottom))
+  )
