File: Pixy-68000/Pixy-68020-0/KiCad/Pixy-68020.kicad_pcb (KiCad board)
At the start: 4 copper layers, 0 parts

Commit message: Fixed minor footprint issue.
Parts:
- added ?: , , F.Cu at (169.1, 38.0)
- added ?: , , F.Cu at (39.1, 147.9)
- added ?: , , F.Cu at (169.1, 147.9)
- added REF**: HandCraft_MountingHole_3mm_Pad, KiCad_Library:HandCraft_MountingHole_3mm_Pad, F.Cu at (39.1, 147.9)
- added REF**: HandCraft_MountingHole_3mm_Pad, KiCad_Library:HandCraft_MountingHole_3mm_Pad, F.Cu at (169.1, 38.0)
- added REF**: HandCraft_MountingHole_3mm_Pad, KiCad_Library:HandCraft_MountingHole_3mm_Pad, F.Cu at (169.1, 147.9)
- added REF**: HandCraft_MountingHole_3mm_Pad, KiCad_Library:HandCraft_MountingHole_3mm_Pad, F.Cu at (39.1, 38.0)
Other:
- board outline added: 140 x 120 mm

Commit message: WIP
Parts:
- added BT1: ML2032, KiCad_Library:BatteryHolder_Keystone_103_1x20mm, F.Cu at (137.7, 60.2)
- added C1: 0.1u, KiCad_Library:C_0805_2012, F.Cu at (212.9, 24.2)
- added C10: 0.1u, KiCad_Library:C_0805_2012, F.Cu at (104.4, 127.6)
- added C11: 0.1u, KiCad_Library:C_0805_2012, F.Cu at (91.6, 136.3)
- added C12: 0.1u, KiCad_Library:C_0805_2012, F.Cu at (117.8, 128.3)
- added C13: 0.1u, KiCad_Library:C_0805_2012, F.Cu at (119.9, 130.4)
- added C14: 0.1u, KiCad_Library:C_0805_2012, F.Cu at (129.8, 129.9)
- added C15: 0.1u, KiCad_Library:C_0805_2012, F.Cu at (114.2, 110.2)
- added C16: 0.1u, KiCad_Library:C_0805_2012, F.Cu at (118.9, 110.2)
- added C17: 0.1u, KiCad_Library:C_0805_2012, F.Cu at (128.8, 110.8)
- added C18: 0.1u, KiCad_Library:C_0805_2012, F.Cu at (134.3, 110.8)
- added C19: 0.1u, KiCad_Library:C_0805_2012, F.Cu at (104.5, 110.4)
- added C2: 100u, KiCad_Library:CP_Radial_D5.0mm_P2.50mm, F.Cu at (252.3, 30.9)
- added C20: 0.1u, KiCad_Library:C_0805_2012, F.Cu at (81.9, 104.3)
- added C21: 0.1u, KiCad_Library:C_0805_2012, F.Cu at (219.8, 42.7)
- added C22: 0.1u, KiCad_Library:C_0805_2012, F.Cu at (219.8, 45.7)
- added C23: 0.1u, KiCad_Library:C_0805_2012, F.Cu at (219.8, 48.7)
- added C24: 0.1u, KiCad_Library:C_0805_2012, F.Cu at (219.8, 51.7)
- added C25: 0.1u, KiCad_Library:C_0805_2012, F.Cu at (219.8, 54.7)
- added C26: 0.1u, KiCad_Library:C_0805_2012, F.Cu at (219.8, 57.7)
- added C27: 0.1u, KiCad_Library:C_0805_2012, F.Cu at (219.8, 60.7)
- added C28: 0.1u, KiCad_Library:C_0805_2012, F.Cu at (224.6, 27.6)
- added C29: 0.1u, KiCad_Library:C_0805_2012, F.Cu at (224.6, 30.6)
- added C3: TPSA106K010R0900, KiCad_Library:CAPMP3216X166, F.Cu at (32.0, 31.7)
- added C30: TPSA106K010R0900, KiCad_Library:CAPMP3216X166, F.Cu at (32.0, 35.0)
- added C31: 0.1u, KiCad_Library:C_0805_2012, F.Cu at (224.6, 33.6)
- added C32: 0.1u, KiCad_Library:C_0805_2012, F.Cu at (224.6, 36.6)
- added C33: 0.1u, KiCad_Library:C_0805_2012, F.Cu at (224.6, 39.7)
- added C34: 0.1u, KiCad_Library:C_0805_2012, F.Cu at (224.6, 42.7)
- added C35: 0.1u, KiCad_Library:C_0805_2012, F.Cu at (224.6, 45.7)
- added C36: 0.1u, KiCad_Library:C_0805_2012, F.Cu at (224.6, 48.7)
- added C37: 0.1u, KiCad_Library:C_0805_2012, F.Cu at (224.6, 51.7)
- added C38: 0.1u, KiCad_Library:C_0805_2012, F.Cu at (224.6, 54.7)
- added C39: 0.1u, KiCad_Library:C_0805_2012, F.Cu at (224.6, 57.7)
- added C4: 0.1u, KiCad_Library:C_0805_2012, F.Cu at (215.0, 30.6)
- added C40: 10u, KiCad_Library:CP_Radial_D5.0mm_P2.50mm, F.Cu at (252.3, 44.0)
- added C41: 0.1u, KiCad_Library:C_0805_2012, F.Cu at (224.6, 60.7)
- added C42: 4u, KiCad_Library:CP_Radial_D5.0mm_P2.50mm, F.Cu at (252.3, 50.6)
- added C43: 0.1u, KiCad_Library:C_0805_2012, F.Cu at (229.4, 27.6)
- added C44: 30p, KiCad_Library:C_0805_2012, F.Cu at (229.4, 30.6)
- added C45: 30p, KiCad_Library:C_0805_2012, F.Cu at (229.4, 33.6)
- added C46: 4u, KiCad_Library:CP_Radial_D5.0mm_P2.50mm, F.Cu at (252.3, 57.1)
- added C47: 0.1u, KiCad_Library:C_0805_2012, F.Cu at (229.4, 36.6)
- added C48: 100u, KiCad_Library:CP_Radial_D5.0mm_P2.50mm, F.Cu at (258.9, 30.9)
- added C49: 6.8p, KiCad_Library:C_0805_2012, F.Cu at (229.4, 39.7)
- added C5: 0.1u, KiCad_Library:C_0805_2012, F.Cu at (114.0, 127.5)
- added C50: 6.8p, KiCad_Library:C_0805_2012, F.Cu at (229.4, 42.7)
- added C51: 10u, KiCad_Library:CP_Radial_D5.0mm_P2.50mm, F.Cu at (258.9, 37.5)
- added C52: 0.1u, KiCad_Library:C_0805_2012, F.Cu at (229.4, 45.7)
- added C53: 0.1u, KiCad_Library:C_0805_2012, F.Cu at (229.4, 48.7)
- added C54: 0.1u, KiCad_Library:C_0805_2012, F.Cu at (229.4, 51.7)
- added C55: 0.1u, KiCad_Library:C_0805_2012, F.Cu at (229.4, 54.7)
- added C56: 0.1u, KiCad_Library:C_0805_2012, F.Cu at (229.4, 57.7)
- added C57: 0.1u, KiCad_Library:C_0805_2012, F.Cu at (229.4, 60.7)
- added C58: 0.1u, KiCad_Library:C_0805_2012, F.Cu at (234.2, 27.6)
- added C59: 0.1u, KiCad_Library:C_0805_2012, F.Cu at (234.2, 30.6)
- added C6: 0.1u, KiCad_Library:C_0805_2012, F.Cu at (214.5, 34.7)
- added C60: 0.1u, KiCad_Library:C_0805_2012, F.Cu at (234.2, 33.6)
- added C61: 0.1u, KiCad_Library:C_0805_2012, F.Cu at (234.2, 36.6)
- added C62: 0.1u, KiCad_Library:C_0805_2012, F.Cu at (234.2, 39.7)
- added C63: 10u, KiCad_Library:CP_Radial_D5.0mm_P2.50mm, F.Cu at (258.9, 44.0)
- added C64: 0.1u, KiCad_Library:C_0805_2012, F.Cu at (234.2, 42.7)
- added C65: 10u, KiCad_Library:C_0805_2012, F.Cu at (234.2, 45.7)
- added C66: 0.1u, KiCad_Library:C_0805_2012, F.Cu at (234.2, 48.7)
- added C67: 10u, KiCad_Library:C_0805_2012, F.Cu at (234.2, 51.7)
- added C68: 100u, KiCad_Library:CP_Radial_D5.0mm_P2.50mm, F.Cu at (258.9, 50.6)
- added C69: 10u, KiCad_Library:C_0805_2012, F.Cu at (234.2, 54.7)
- added C7: 0.1u, KiCad_Library:C_0805_2012, F.Cu at (127.6, 127.3)
- added C70: 10u, KiCad_Library:C_0805_2012, F.Cu at (234.2, 57.7)
- added C71: 100u, KiCad_Library:CP_Radial_D5.0mm_P2.50mm, F.Cu at (258.9, 57.1)
- added C72: 0.1u, KiCad_Library:C_0805_2012, F.Cu at (234.2, 60.7)
- added C73: 0.1u, KiCad_Library:C_0805_2012, F.Cu at (239.0, 27.6)
- added C74: 0.1u, KiCad_Library:C_0805_2012, F.Cu at (239.0, 30.6)
- added C75: 0.1u, KiCad_Library:C_0805_2012, F.Cu at (239.0, 33.6)
- added C76: 0.1u, KiCad_Library:C_0805_2012, F.Cu at (239.0, 36.6)
- added C77: 0.1u, KiCad_Library:C_0805_2012, F.Cu at (239.0, 39.7)
- added C78: 0.1u, KiCad_Library:C_0805_2012, F.Cu at (239.0, 42.7)
- added C79: 0.1u, KiCad_Library:C_0805_2012, F.Cu at (239.0, 45.7)
- added C8: 0.1u, KiCad_Library:C_0805_2012, F.Cu at (135.4, 123.8)
- added C9: 100u, KiCad_Library:CP_Radial_D5.0mm_P2.50mm, F.Cu at (252.3, 37.5)
- added CN1: RS232C, KiCad_Library:DSUB-9_Pins_Horizontal_P2.77x2.84mm_EdgePinOffset4.94mm_Housed_MountingHolesOffset4.94mm, F.Cu at (28.5, 99.9)
- added D1: POWER, KiCad_Library:LED_D3.0mm, F.Cu at (53.5, 26.6)
- added D10: ESD5B5.0ST1G, KiCad_Library:D_SOD-523, F.Cu at (54.1, 42.8)
- added D11: SS14, KiCad_Library:D_SMA, F.Cu at (66.6, 51.6)
- added D12: ESD9B3.3ST5G, KiCad_Library:D_SOD-923, F.Cu at (128.6, 24.1)
- added D13: ESD9B3.3ST5G, KiCad_Library:D_SOD-923, F.Cu at (128.6, 26.0)
- added D14: ESD9B3.3ST5G, KiCad_Library:D_SOD-923, F.Cu at (128.6, 27.9)
- added D15: ESD9B3.3ST5G, KiCad_Library:D_SOD-923, F.Cu at (128.6, 29.9)
- added D16: ESD9B3.3ST5G, KiCad_Library:D_SOD-923, F.Cu at (128.6, 31.9)
- added D17: ESD9B3.3ST5G, KiCad_Library:D_SOD-923, F.Cu at (128.6, 33.8)
- added D18: 1SS367, KiCad_Library:D_SOD-323F, F.Cu at (81.5, 23.7)
- added D19: ESD5B5.0ST1G, KiCad_Library:D_SOD-523, F.Cu at (54.1, 45.2)
- added D2: INIT, KiCad_Library:LED_D3.0mm, F.Cu at (38.4, 129.2)
- added D20: ACT0, KiCad_Library:LED_D3.0mm, F.Cu at (44.6, 134.7)
- added D21: ACT1, KiCad_Library:LED_D3.0mm, F.Cu at (44.5, 140.4)
- added D3: DONE, KiCad_Library:LED_D3.0mm, F.Cu at (38.4, 134.8)
- added D4: RUN, KiCad_Library:LED_D3.0mm, F.Cu at (38.4, 140.3)
- added D5: ESD5B5.0ST1G, KiCad_Library:D_SOD-523, F.Cu at (54.1, 33.0)
- added D6: ESD5B5.0ST1G, KiCad_Library:D_SOD-523, F.Cu at (54.1, 35.4)
- added D7: ESD5B5.0ST1G, KiCad_Library:D_SOD-523, F.Cu at (54.1, 37.9)
- added D8: ESD5B5.0ST1G, KiCad_Library:D_SOD-523, F.Cu at (54.1, 40.3)
- added D9: HALT, KiCad_Library:LED_D3.0mm, F.Cu at (44.4, 129.2)
- added F1: MF-R050, KiCad_Library:Fuse_Bourns_MF-RG300, F.Cu at (57.4, 32.0)
- added J1: USB_C_Receptacle_USB2.0, KiCad_Library:USB_C_Receptacle_HRO_TYPE-C-31-M-12, F.Cu at (43.3, 24.4)
- added J10: Agilent_LA_20, KiCad_Library:PinHeader_2x10_P2.54mm_Vertical, F.Cu at (183.6, 53.7)
- added J11: Agilent_LA_20, KiCad_Library:PinHeader_2x10_P2.54mm_Vertical, F.Cu at (173.4, 53.7)
- added J12: Agilent_LA_20, KiCad_Library:PinHeader_2x10_P2.54mm_Vertical, F.Cu at (193.9, 53.7)
- added J13: Agilent_LA_20, KiCad_Library:PinHeader_2x10_P2.54mm_Vertical, F.Cu at (193.9, 112.5)
- added J14: Agilent_LA_20, KiCad_Library:PinHeader_2x10_P2.54mm_Vertical, F.Cu at (183.6, 112.5)
- added J15: Agilent_LA_20, KiCad_Library:PinHeader_2x10_P2.54mm_Vertical, F.Cu at (173.4, 112.5)
- added J16: Agilent_LA_20, KiCad_Library:PinHeader_2x10_P2.54mm_Vertical, F.Cu at (163.2, 112.5)
- added J2: USB_C_Receptacle_USB2.0_HOST, KiCad_Library:USB_C_Receptacle_HRO_TYPE-C-31-M-12, F.Cu at (66.6, 24.4)
- added J3: Micro_TF_Card, KiCad_Library:Hirose_DM3D-SF, F.Cu at (116.9, 28.7)
- added J4: Agilent_LA_20, KiCad_Library:PinHeader_2x10_P2.54mm_Vertical, F.Cu at (163.2, 83.1)
- added J5: Agilent_LA_20, KiCad_Library:PinHeader_2x10_P2.54mm_Vertical, F.Cu at (173.4, 83.1)
- added J6: SNDL, KiCad_Library:CUI_RCJ-042, F.Cu at (20.3, 56.2)
- added J7: SNDR, KiCad_Library:CUI_RCJ-042, F.Cu at (20.3, 44.1)
- added J8: Agilent_LA_20, KiCad_Library:PinHeader_2x10_P2.54mm_Vertical, F.Cu at (193.9, 83.1)
- added J9: Agilent_LA_20, KiCad_Library:PinHeader_2x10_P2.54mm_Vertical, F.Cu at (183.6, 83.1)
- added JP1: CHARGE, KiCad_Library:SolderJumper-2_P1.3mm_Open_RoundedPad1.0x1.5mm, F.Cu at (77.1, 24.0)
- added L1: 1k@100M 0.8A, KiCad_Library:L_0603_1608, F.Cu at (46.6, 65.3)
- added L2: 1k@100M 0.8A, KiCad_Library:L_0603_1608, F.Cu at (46.6, 61.2)
- added L3: 1k@100M 2A, KiCad_Library:L_1206_3216, F.Cu at (67.0, 34.4)
- added L4: 1k@100M 2A, KiCad_Library:L_1206_3216, F.Cu at (67.0, 37.7)
- added L5: 1k@100M 2A, KiCad_Library:L_1206_3216, F.Cu at (67.0, 41.1)
- added L6: 1k@100M 2A, KiCad_Library:L_1206_3216, F.Cu at (67.0, 44.4)
- added LCD1: SLGM320240F, KiCad_Library:PinHeader_1x20_P2.54mm_Vertical, F.Cu at (140.4, 24.7)
- added R1: 2k, KiCad_Library:R_0805_2012, F.Cu at (219.4, 70.0)
- added R10: 2k, KiCad_Library:R_0805_2012, F.Cu at (219.4, 96.5)
- added R11: 5.1k, KiCad_Library:R_0805_2012, F.Cu at (224.2, 70.0)
- added R12: 1.5k, KiCad_Library:R_0805_2012, F.Cu at (224.2, 72.9)
- added R13: 5.1k, KiCad_Library:R_0805_2012, F.Cu at (224.2, 75.9)
- added R14: 12k, KiCad_Library:R_0805_2012, F.Cu at (224.2, 78.8)
- added R15: 10k, KiCad_Library:R_0805_2012, F.Cu at (224.2, 81.8)
- added R16: 10k, KiCad_Library:R_0805_2012, F.Cu at (224.2, 84.7)
- added R17: 5.1k, KiCad_Library:R_0805_2012, F.Cu at (224.2, 87.7)
- added R18: 10k, KiCad_Library:R_0805_2012, F.Cu at (224.2, 90.6)
- added R19: 10k, KiCad_Library:R_0805_2012, F.Cu at (224.2, 93.6)
- added R2: 5.1k, KiCad_Library:R_0805_2012, F.Cu at (219.4, 72.9)
- added R20: 10k, KiCad_Library:R_0805_2012, F.Cu at (224.2, 96.5)
- added R21: 2.2k, KiCad_Library:R_0805_2012, F.Cu at (228.9, 70.0)
- added R22: 10k, KiCad_Library:R_0805_2012, F.Cu at (228.9, 72.9)
- added R23: 10k, KiCad_Library:R_0805_2012, F.Cu at (228.9, 75.9)
- added R24: 1.5k, KiCad_Library:R_0805_2012, F.Cu at (228.9, 78.8)
- added R25: 10k, KiCad_Library:R_0805_2012, F.Cu at (228.9, 81.8)
- added R26: 10k, KiCad_Library:R_0805_2012, F.Cu at (228.9, 84.7)
- added R27: 10k, KiCad_Library:R_0805_2012, F.Cu at (228.9, 87.7)
- added R28: 10k, KiCad_Library:R_0805_2012, F.Cu at (228.9, 90.6)
- added R29: 10k, KiCad_Library:R_0805_2012, F.Cu at (228.9, 93.6)
- added R3: 5.1k, KiCad_Library:R_0805_2012, F.Cu at (219.4, 75.9)
- added R30: 4.7k, KiCad_Library:R_0805_2012, F.Cu at (228.9, 96.5)
- added R31: 4.7k, KiCad_Library:R_0805_2012, F.Cu at (233.7, 70.0)
- added R32: 4.7k, KiCad_Library:R_0805_2012, F.Cu at (233.7, 72.9)
- added R33: 2k, KiCad_Library:R_0805_2012, F.Cu at (233.7, 75.9)
- added R34: 10k, KiCad_Library:R_0805_2012, F.Cu at (233.7, 78.8)
- added R35: 10k, KiCad_Library:R_0805_2012, F.Cu at (233.7, 81.8)
- added R36: 10k, KiCad_Library:R_0805_2012, F.Cu at (233.7, 84.7)
- added R37: 2k, KiCad_Library:R_0805_2012, F.Cu at (233.7, 87.7)
- added R38: 2k, KiCad_Library:R_0805_2012, F.Cu at (233.7, 90.6)
- added R39: 1k, KiCad_Library:R_0805_2012, F.Cu at (128.1, 38.0)
- added R4: 5.1k, KiCad_Library:R_0805_2012, F.Cu at (219.4, 78.8)
- added R40: 4.7k, KiCad_Library:R_0805_2012, F.Cu at (233.7, 93.6)
- added R41: 4.7k, KiCad_Library:R_0805_2012, F.Cu at (233.7, 96.5)
- added R42: 10k, KiCad_Library:R_0805_2012, F.Cu at (238.4, 70.0)
- added R43: 4.7k, KiCad_Library:R_0805_2012, F.Cu at (238.4, 72.9)
- added R44: 4.7k, KiCad_Library:R_0805_2012, F.Cu at (238.4, 75.9)
- added R45: 47, KiCad_Library:R_0805_2012, F.Cu at (238.4, 78.8)
- added R46: 10k, KiCad_Library:R_0805_2012, F.Cu at (238.4, 81.8)
- added R47: 47, KiCad_Library:R_0805_2012, F.Cu at (238.4, 84.7)
- added R48: 4.7k, KiCad_Library:R_0805_2012, F.Cu at (238.4, 87.7)
- added R49: 4.7k, KiCad_Library:R_0805_2012, F.Cu at (238.4, 90.6)
- added R5: 5.1k, KiCad_Library:R_0805_2012, F.Cu at (219.4, 81.8)
- added R50: 4.7k, KiCad_Library:R_0805_2012, F.Cu at (238.4, 93.6)
- added R51: 4.7k, KiCad_Library:R_0805_2012, F.Cu at (238.4, 96.5)
- added R6: 2k, KiCad_Library:R_0805_2012, F.Cu at (219.4, 84.7)
- added R7: 2.2k, KiCad_Library:R_0805_2012, F.Cu at (219.4, 87.7)
- added R8: 2k, KiCad_Library:R_0805_2012, F.Cu at (219.4, 90.6)
- added R9: 2k, KiCad_Library:R_0805_2012, F.Cu at (219.4, 93.6)
- added SW1: RESET, KiCad_Library:TactSwitch, F.Cu at (59.5, 137.2)
- added U1: LT1963AEST, KiCad_Library:SOT-223-3_TabPin2, F.Cu at (42.2, 37.3)
- added U10: 93LC56BT-I, KiCad_Library:MSOP-8_3x3mm_P0.65mm, F.Cu at (53.9, 53.9)
- added U11: NJM4558DD, KiCad_Library:DIP-8_W7.62mm, F.Cu at (27.5, 67.7)
- added U12: BU9480F, KiCad_Library:SOP-8_3.9x4.9mm_P1.27mm, F.Cu at (31.6, 83.4)
- added U13: SC28L92A1B, KiCad_Library:SOT307-2_NXP-M, F.Cu at (61.4, 103.4)
- added U14: TRS3232EIDR, KiCad_Library:SOIC-16_3.9x9.9mm_P1.27mm, F.Cu at (43.8, 112.0)
- added U15: TRS3232EIDR, KiCad_Library:SOIC-16_3.9x9.9mm_P1.27mm, F.Cu at (43.9, 97.8)
- added U2: LCMXO2-1200UHC/2000HC-4FTG256C, KiCad_Library:LCMXO2-FTG256, F.Cu at (93.8, 118.8)
- added U3: MC68EC020FG25, KiCad_Library:MC68EC020FG25, F.Cu at (112.5, 81.6)
- added U4: LT1963AEST, KiCad_Library:SOT-223-3_TabPin2, F.Cu at (42.2, 45.6)
- added U5: AS4C4M32SA, KiCad_Library:SOIC-86, F.Cu at (123.0, 119.2)
- added U6: ESP32-S3-MINI-1-N8, KiCad_Library:ESP32-S3-MINI-1_EXP, F.Cu at (95.7, 30.8)
- added U7: MCP7940N-xMS, KiCad_Library:MSOP-8_3x3mm_P0.65mm, F.Cu at (79.4, 29.2)
- added U8: BC848CDW1T1G, KiCad_Library:SOT65P210X110-6N, F.Cu at (73.2, 69.1)
- added U9: FT4232H, KiCad_Library:LQFP-64_10x10mm_P0.5mm, F.Cu at (59.9, 69.7)
- added X1: ASE-25MHz, KiCad_Library:Oscillator_SMD_Abracon_ASE-4Pin_3.2x2.5mm_HandSoldering, F.Cu at (82.0, 100.7)
- added X2: ASE-24.576MHz, KiCad_Library:Oscillator_SMD_Abracon_ASE-4Pin_3.2x2.5mm_HandSoldering, F.Cu at (91.5, 132.7)
- added Y1: 12MHz, KiCad_Library:Crystal_HC18-U_Vertical, F.Cu at (37.5, 60.9)
- added Y2: 32.768k, KiCad_Library:Crystal_HC18-U_Vertical, F.Cu at (78.9, 41.9)
- moved ? 32.5 mm to (199.1, 25.4)
- moved REF** 32.5 mm to (199.1, 25.4)
- moved ? 30.4 mm to (199.1, 142.9)
- moved REF** 30.4 mm to (199.1, 142.9)
- moved REF** 18.6 mm to (25.3, 25.4)
- moved ? 14.6 mm to (25.3, 142.9)
- moved REF** 14.6 mm to (25.3, 142.9)
Routing:
- net VCC: track 0.00 -> 137.4 mm, vias 0 -> 36
- net /SD7: track 0.00 -> 128.0 mm, vias 0 -> 2
- net /SD5: track 0.00 -> 125.4 mm, vias 0 -> 3
- net /SD3: track 0.00 -> 125.3 mm, vias 0 -> 2
- net /SD6: track 0.00 -> 119.7 mm, vias 0 -> 4
- net /SD9: track 0.00 -> 118.4 mm, vias 0 -> 3
- net /SD11: track 0.00 -> 118.1 mm, vias 0 -> 4
- net /SD1: track 0.00 -> 117.1 mm, vias 0 -> 2
- net /SD8: track 0.00 -> 117.1 mm, vias 0 -> 5
- net /SD4: track 0.00 -> 115.9 mm, vias 0 -> 3
- net /SD10: track 0.00 -> 115.7 mm, vias 0 -> 2
- net /SD14: track 0.00 -> 115.1 mm, vias 0 -> 2
- net /SD23: track 0.00 -> 114.9 mm, vias 0 -> 4
- net /SD13: track 0.00 -> 114.8 mm, vias 0 -> 3
- net /SD15: track 0.00 -> 114.2 mm, vias 0 -> 1
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- added copper zone on B.Cu, net GND
- added copper zone on F.Cu, net GND
- added copper zone on In2.Cu, net GND
- added copper zone on In1.Cu, net VCC
Other:
- board size 140 x 120 mm -> 183.7 x 127.6 mm
