File: Pixy-68000/Pixy-68020-0/KiCad/Pixy-68020.kicad_sch (KiCad schematic)
At the start: 197 parts, among them CN1 RS232C, J1 USB_C_Receptacle_USB2.0, J10 Agilent_LA_20, J11 Agilent_LA_20, J12 Agilent_LA_20, J13 Agilent_LA_20, J14 Agilent_LA_20, J15 Agilent_LA_20, J16 Agilent_LA_20, J2 USB_C_Receptacle_USB2.0_HOST, J3 Micro_TF_Card, J4 Agilent_LA_20, J5 Agilent_LA_20, J6 SNDL, J7 SNDR, J8 Agilent_LA_20, J9 Agilent_LA_20, SW1 RESET, U1 LT1963AEST, U10 93LC56BT-I, U11 NJM4558DD, U12 BU9480F, U13 SC28L92A1B, U14 TRS3232EIDR, U15 TRS3232EIDR, U2 LCMXO2-1200UHC/2000HC-4FTG256C, U3 MC68EC020FG25, U4 LT1963AEST, U5 AS4C4M32SA, U6 ESP32-S3-MINI-1-N8, U7 MCP7940N-xMS, U8 BC848CDW1T1G, U9 FT4232H, X1 ASE-25MHz, X2 ASE-24.576MHz, Y1 12MHz, Y2 32.768k

Commit message: Changed MachXO2 footprint.
Parts:
- U2: footprint KiCad_Library:LCMXO2-FTG256 -> KiCad_Library:LCMXO2-FTG256_LandOut
Changed lines of the file:
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@@
 			)
 		)
-		(property "Footprint" "KiCad_Library:LCMXO2-FTG256"
+		(property "Footprint" "KiCad_Library:LCMXO2-FTG256_LandOut"
 			(at 228.092 179.324 0)
 			(effects
@@
 			)
 		)
-		(property "Footprint" "KiCad_Library:LCMXO2-FTG256"
+		(property "Footprint" "KiCad_Library:LCMXO2-FTG256_LandOut"
 			(at 176.022 179.324 0)
 			(effects
@@
 			)
 		)
-		(property "Footprint" "KiCad_Library:LCMXO2-FTG256"
+		(property "Footprint" "KiCad_Library:LCMXO2-FTG256_LandOut"
 			(at 489.712 448.564 0)
 			(effects
@@
 			)
 		)
-		(property "Footprint" "KiCad_Library:LCMXO2-FTG256"
+		(property "Footprint" "KiCad_Library:LCMXO2-FTG256_LandOut"
 			(at 123.952 179.324 0)
 			(effects
@@
 			)
 		)
-		(property "Footprint" "KiCad_Library:LCMXO2-FTG256"
+		(property "Footprint" "KiCad_Library:LCMXO2-FTG256_LandOut"
 			(at 280.162 237.744 0)
 			(effects
@@
 			)
 		)
-		(property "Footprint" "KiCad_Library:LCMXO2-FTG256"
+		(property "Footprint" "KiCad_Library:LCMXO2-FTG256_LandOut"
 			(at 280.162 297.434 0)
 			(effects
@@
 			)
 		)
-		(property "Footprint" "KiCad_Library:LCMXO2-FTG256"
+		(property "Footprint" "KiCad_Library:LCMXO2-FTG256_LandOut"
 			(at 280.162 179.324 0)
 			(effects

Commit message: Fixed minor footprint issue.
Parts:
- C3, C30: footprint TPSA106K010R0900:CAPMP3216X166 -> KiCad_Library:CAPMP3216X166
- J1, J2: footprint kekyo:USB_C_Receptacle_HRO_TYPE-C-31-M-12 -> KiCad_Library:USB_C_Receptacle_HRO_TYPE-C-31-M-12
- J6, J7: footprint (none) -> KiCad_Library:CUI_RCJ-042
- U11: footprint (none) -> KiCad_Library:DIP-8_W7.62mm
- U13: footprint kekyo:SOT307-2_NXP-M -> KiCad_Library:SOT307-2_NXP-M
- U8: footprint BC848CDW1T1G:SOT65P210X110-6N -> KiCad_Library:SOT65P210X110-6N
- U9: footprint (none) -> KiCad_Library:LQFP-64_10x10mm_P0.5mm
Changed lines of the file:
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@@
 			)
 		)
-		(property "Footprint" ""
+		(property "Footprint" "KiCad_Library:LQFP-64_10x10mm_P0.5mm"
 			(at 115.57 304.8 0)
 			(effects
@@
 			)
 		)
-		(property "Footprint" "kekyo:USB_C_Receptacle_HRO_TYPE-C-31-M-12"
+		(property "Footprint" "KiCad_Library:USB_C_Receptacle_HRO_TYPE-C-31-M-12"
 			(at 27.686 405.892 0)
 			(effects
@@
 			)
 		)
-		(property "Footprint" "TPSA106K010R0900:CAPMP3216X166"
+		(property "Footprint" "KiCad_Library:CAPMP3216X166"
 			(at 137.16 355.6 0)
 			(effects
@@
 			)
 		)
-		(property "Footprint" ""
+		(property "Footprint" "KiCad_Library:DIP-8_W7.62mm"
 			(at 321.31 353.06 0)
 			(effects
@@
 			)
 		)
-		(property "Footprint" "TPSA106K010R0900:CAPMP3216X166"
+		(property "Footprint" "KiCad_Library:CAPMP3216X166"
 			(at 147.32 382.27 0)
 			(effects
@@
 			)
 		)
-		(property "Footprint" "BC848CDW1T1G:SOT65P210X110-6N"
+		(property "Footprint" "KiCad_Library:SOT65P210X110-6N"
 			(at 322.58 297.18 0)
 			(effects
@@
 			)
 		)
-		(property "Footprint" ""
+		(property "Footprint" "KiCad_Library:CUI_RCJ-042"
 			(at 443.23 322.58 0)
 			(effects
@@
 			)
 		)
-		(property "Footprint" ""
+		(property "Footprint" "KiCad_Library:CUI_RCJ-042"
 			(at 443.23 345.44 0)
 			(effects
@@
 			)
 		)
-		(property "Footprint" "BC848CDW1T1G:SOT65P210X110-6N"
+		(property "Footprint" "KiCad_Library:SOT65P210X110-6N"
 			(at 322.58 280.67 0)
 			(effects
@@
 			)
 		)
-		(property "Footprint" "kekyo:USB_C_Receptacle_HRO_TYPE-C-31-M-12"
+		(property "Footprint" "KiCad_Library:USB_C_Receptacle_HRO_TYPE-C-31-M-12"
 			(at 27.686 290.322 0)
 			(effects
@@
 			)
 		)
-		(property "Footprint" "kekyo:SOT307-2_NXP-M"
+		(property "Footprint" "KiCad_Library:SOT307-2_NXP-M"
 			(at 383.286 108.966 0)
 			(effects
@@
 			)
 		)
-		(property "Footprint" ""
+		(property "Footprint" "KiCad_Library:DIP-8_W7.62mm"
 			(at 400.05 345.44 0)
 			(effects
@@
 			)
 		)
-		(property "Footprint" ""
+		(property "Footprint" "KiCad_Library:DIP-8_W7.62mm"
 			(at 400.05 322.58 0)
 			(effects

Commit message: WIP
Parts:
- added R39: 1k, KiCad_Library:R_0805_2012, symbol Device:R
- LCD1: footprint KiCad_Library:PinHeader_1x08_P2.54mm_Vertical -> KiCad_Library:PinHeader_1x20_P2.54mm_Vertical
- U2: footprint KiCad_Library:LCMXO2-FTG256_LandOut -> KiCad_Library:LCMXO2-FTG256
- U6: footprint ESP32-S3-MINI-1_EXP -> KiCad_Library:ESP32-S3-MINI-1_EXP
Connections:
- net GND: now also J3.10 (SW2), J3.11 (SHIELD); no longer J3.9 (SHIELD)
- net VCCESP: now also R39.2
- net /TFRDY: now reaches U6.41 (IO45)
- net /TFRDY: now also J3.9 (SW1), R39.1
- no-connect marks 79 -> 78
Other:
- moved on the sheet: C32, C48, D12, D13, D14, D15, D16, D17
